File: src/kicad/triplejump.kicad_pcb (KiCad board)
At the start: 2 copper layers, 340 x 112 mm, 26 parts, among them M3 MountingHole_3.2mm_M3, SW1 SW_Push_45deg, SW10 SW_Push_45deg, SW11 SW_Push_45deg, SW12 SW_Push_45deg, SW13 SW_Push_45deg, SW14 SW_Push_45deg, SW15 SW_Push_45deg, SW16 SW_Push_45deg, SW17 SW_Push_45deg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

Commit message: Updated PCB (and gerbers) to fix subtle UP 1 missalignment; remove one NPTH
Parts:
- removed the M3 at (192.0, 78.0)
- moved SW8 0.30 mm to (85.8, 37.8)
Changed lines of the file:
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@@
       (net 1 "GND") (pinfunction "2") (pintype "passive"))
-  )
-  (footprint "MountingHole:MountingHole_3.2mm_M3" (layer "F.Cu")
-    (at 192 78)
-    (descr "Mounting Hole 3.2mm, no annular, M3")
-    (tags "mounting hole 3.2mm no annular m3")
-    (attr exclude_from_pos_files exclude_from_bom)
-    (fp_text reference "M3" (at 0 -4.2) (layer "B.SilkS")
-        (effects (font (size 1 1) (thickness 0.15)) (justify mirror))
-    )
-    (fp_text value "MountingHole_3.2mm_M3" (at 0 4.2) (layer "F.Fab")
-        (effects (font (size 1 1) (thickness 0.15)))
-    )
-    (fp_text user "${REFERENCE}" (at 0 0) (layer "F.Fab")
-        (effects (font (size 1 1) (thickness 0.15)))
-    )
-    (fp_circle (center 0 0) (end 3.2 0)
-      (stroke (width 0.15) (type solid)) (fill none) (layer "Cmts.User"))
-    (fp_circle (center 0 0) (end 3.45 0)
-      (stroke (width 0.05) (type solid)) (fill none) (layer "F.CrtYd"))
-    (pad "" np_thru_hole circle (at 0 0) (size 3.2 3.2) (drill 3.2) (layers "*.Cu" "*.Mask"))
   )
   (footprint "Button_Switch_THT:SW_PUSH_6mm" locked (layer "F.Cu")
@@
       (net 1 "GND") (pinfunction "2") (pintype "passive"))
   )
-  (footprint "keyswitches.pretty-master:Kailh_socket_PG1350" locked (layer "F.Cu")
-    (at 86.050878 37.872337 -24)
+  (footprint "keyswitches.pretty-master:Kailh_socket_PG1350" (layer "F.Cu")
+    (at 85.778956 37.751269 -24)
     (descr "Kailh \"Choc\" PG1350 keyswitch socket mount")
     (tags "kailh,choc")
@@
     (fp_line (start 7.5 7.5) (end -7.5 7.5)
       (stroke (width 0.15) (type solid)) (layer "F.Fab"))
-    (pad "" np_thru_hole circle locked (at -5.5 0 336) (size 1.7018 1.7018) (drill 1.7018) (layers "*.Cu" "*.Mask"))
-    (pad "" np_thru_hole circle locked (at -5 3.75 336) (size 3 3) (drill 3) (layers "*.Cu" "*.Mask"))
-    (pad "" np_thru_hole circle locked (at 0 0 336) (size 3.429 3.429) (drill 3.429) (layers "*.Cu" "*.Mask"))
-    (pad "" np_thru_hole circle locked (at 0 5.95 336) (size 3 3) (drill 3) (layers "*.Cu" "*.Mask"))
-    (pad "" np_thru_hole circle locked (at 5.22 -4.2 336) (size 0.9906 0.9906) (drill 0.9906) (layers "*.Cu" "*.Mask"))
-    (pad "" np_thru_hole circle locked (at 5.5 0 336) (size 1.7018 1.7018) (drill 1.7018) (layers "*.Cu" "*.Mask"))
-    (pad "1" smd rect locked (at 3.275 5.95 336) (size 2.6 2.6) (layers "B.Cu" "B.Paste" "B.Mask")
+    (pad "" np_thru_hole circle (at -5.5 0 336) (size 1.7018 1.7018) (drill 1.7018) (layers "*.Cu" "*.Mask"))
+    (pad "" np_thru_hole circle (at -5 3.75 336) (size 3 3) (drill 3) (layers "*.Cu" "*.Mask"))
+    (pad "" np_thru_hole circle (at 0 0 336) (size 3.429 3.429) (drill 3.429) (layers "*.Cu" "*.Mask"))
+    (pad "" np_thru_hole circle (at 0 5.95 336) (size 3 3) (drill 3) (layers "*.Cu" "*.Mask"))
+    (pad "" np_thru_hole circle (at 5.22 -4.2 336) (size 0.9906 0.9906) (drill 0.9906) (layers "*.Cu" "*.Mask"))
+    (pad "" np_thru_hole circle (at 5.5 0 336) (size 1.7018 1.7018) (drill 1.7018) (layers "*.Cu" "*.Mask"))
+    (pad "1" smd rect (at 3.275 5.95 336) (size 2.6 2.6) (layers "B.Cu" "B.Paste" "B.Mask")
       (net 11 "UP") (pinfunction "1") (pintype "passive"))
-    (pad "2" smd rect locked (at -8.275 3.75 336) (size 2.6 2.6) (layers "B.Cu" "B.Paste" "B.Mask")
+    (pad "2" smd rect (at -8.275 3.75 336) (size 2.6 2.6) (layers "B.Cu" "B.Paste" "B.Mask")
       (net 1 "GND") (pinfunction "2") (pintype "passive"))
   )
@@
     (effects (font (size 1 1) (thickness 0.15)) (justify bottom))
   )
-  (gr_text "UP 1" (at 89.81875 30.2 336) (layer "F.SilkS")
+  (gr_text "UP 1" (at 89.546828 30.078932 -24) (layer "F.SilkS")
     (effects (font (size 1 1) (thickness 0.15)) (justify bottom))
   )
